Commit message: feat : new urdf

File: src/cartographer_ros/cartographer_ros/urdf/mid360_backup.urdf (robot description, URDF)
Before this commit: robot mid360, 3 links, 2 joints
Joints:
- joint imu_link_joint: origin xyz=1.22 0.49 0.7 rpy=0 0 0.78 -> xyz=0.76 0.49 0.7 rpy=0 0 0.78
- joint lidar_link_joint: origin xyz=1.22 0.49 0.7 rpy=0 0 0.78 -> xyz=0.76 0.49 0.7 rpy=0 0 0.78
