Commit message: feat : remove imu

File: src/cartographer_ros/cartographer_ros/urdf/mid360.urdf (robot description, URDF)
Before this commit: robot mid360, 3 links, 2 joints
Links:
- link base_link: geometry visual box size=1.52 0.98 1.4
Joints:
- joint imu_link_joint: origin xyz=0.0 0.0 0.0 rpy=0.0 0.0 0.0 -> xyz=0.76 0.49 0.7 rpy=0 0 0.78
- joint lidar_link_joint: origin xyz=0.0 0.0 0.0 rpy=0.0 0.0 0.0 -> xyz=0.76 0.49 0.7 rpy=0 0 0.78

Commit message: chore: lidar height

File: src/cartographer_ros/cartographer_ros/urdf/mid360.urdf (robot description, URDF)
Before this commit: robot mid360, 3 links, 2 joints
Joints:
- joint imu_link_joint: origin xyz=1.22 0.49 0.7 rpy=0 0 0.78 -> xyz=1.22 0.49 0.6 rpy=0 0 0.78
- joint lidar_link_joint: origin xyz=1.22 0.49 0.7 rpy=0 0 0.78 -> xyz=1.22 0.49 0.6 rpy=0 0 0.78

Commit message: feat : add urdf

File: src/cartographer_ros/cartographer_ros/urdf/mid360.urdf (robot description, URDF)
Before this commit: robot mid360, 3 links, 2 joints
Links:
- link base_link: geometry visual box size=1.61 1.0266 1.4265
Joints:
- joint imu_link_joint: origin xyz=1.22 0.49 0.6 rpy=0 0 0.78 -> xyz=1.334265 0.5133 0.61995 rpy=0 0 0.785398
- joint lidar_link_joint: origin xyz=1.22 0.49 0.6 rpy=0 0 0.78 -> xyz=1.334265 0.5133 0.61995 rpy=0 0 0.785398

File: src/cartographer_ros/cartographer_ros/urdf/mid360_backup.urdf (robot description, URDF)
Before this commit: robot mid360, 3 links, 2 joints
Joints:
- joint imu_link_joint: origin xyz=0.76 0.49 0.7 rpy=0 0 0.78 -> xyz=1.22 0.49 0.6 rpy=0 0 0.78
- joint lidar_link_joint: origin xyz=0.76 0.49 0.7 rpy=0 0 0.78 -> xyz=1.22 0.49 0.6 rpy=0 0 0.78

Commit message: feat : modify urdf by CAD

File: src/cartographer_ros/cartographer_ros/urdf/mid360.urdf (robot description, URDF)
Before this commit: robot mid360, 3 links, 2 joints
Joints:
- joint imu_link_joint: origin xyz=1.334265 0.5133 0.61995 rpy=0 0 0.785398 -> xyz=1.29753 0.5133 0.57482 rpy=0 0 0.785398
- joint lidar_link_joint: origin xyz=1.334265 0.5133 0.61995 rpy=0 0 0.785398 -> xyz=1.29753 0.5133 0.57482 rpy=0 0 0.785398
