Commit message: feat : huaian

File: src/cartographer_ros/cartographer_ros/urdf/mid360_nanjing.urdf (robot description, URDF)
Before this commit: robot mid360, 3 links, 2 joints
Joints:
- joint imu_link_joint: origin xyz=1.31753 0.5333 0.42675 rpy=0 0 0.785398 -> xyz=1.29753 0.5133 0.57482 rpy=0 0 0.785398
- joint lidar_link_joint: origin xyz=1.31753 0.5333 0.42675 rpy=0 0 0.785398 -> xyz=1.29753 0.5133 0.57482 rpy=0 0 0.785398

Commit message: feat : add launch

File: src/cartographer_ros/cartographer_ros/urdf/mid360_nanjing.urdf (robot description, URDF)
Before this commit: robot mid360, 3 links, 2 joints
Joints:
- joint imu_link_joint: origin xyz=1.29753 0.5133 0.57482 rpy=0 0 0.785398 -> xyz=1.31753 0.5333 0.57482 rpy=0 0 0.785398
- joint lidar_link_joint: origin xyz=1.29753 0.5133 0.57482 rpy=0 0 0.785398 -> xyz=1.31753 0.5333 0.57482 rpy=0 0 0.785398

Commit message: feat: add a lot

File: src/cartographer_ros/cartographer_ros/urdf/mid360_nanjing.urdf (robot description, URDF)
Before this commit: robot mid360, 3 links, 2 joints
Links:
- added link fore_153; visual box size=0.06 0.04 0.02
- added link lidar_fore; visual box size=0.06 0.04 0.02
- added link livox_frame_192_168_1_153; visual box size=0.06 0.04 0.02
- added link livox_frame_192_168_1_196; visual box size=0.06 0.04 0.02
- added link utm; visual box size=0.06 0.04 0.02
Joints:
- added joint fore_153_joint: type fixed, parent livox_frame_192_168_1_153, child fore_153, origin xyz=0 0 0  rpy= 3.1415926 0 -2.3561944 
- added joint lidar_fore_joint: type fixed, parent lidar_link, child lidar_fore, origin xyz=0 0 0 rpy=0 0 -0.785398
- added joint livox_frame_192_168_1_153_joint: type fixed, parent livox_frame_192_168_1_196, child livox_frame_192_168_1_153, origin xyz=-1.87842 -0.434706 -0.00151078 rpy= 0.000994 0.04232 3.12432  
- added joint livox_frame_192_168_1_196_joint: type fixed, parent base_link, child livox_frame_192_168_1_196, origin xyz=1.31753 0.5333 0.57482 rpy=3.1415926 0 0.785398
- added joint utm_joint: type fixed, parent lidar_fore, child utm, origin xyz=-0.18 -0.51 0.18 rpy=0 0 0

Commit message: feat: carto 20250925

File: src/cartographer_ros/cartographer_ros/urdf/mid360_nanjing.urdf (robot description, URDF)
Before this commit: robot mid360, 8 links, 7 joints
Links:
- removed link utm
- added link gps; visual box size=0.06 0.04 0.02
Joints:
- removed joint utm_joint
- added joint gps_joint: type fixed, parent lidar_fore, child gps, origin xyz=-0.18 -0.51 0.18 rpy=0 0 0

Commit message: 20251217

File: src/cartographer_ros/cartographer_ros/urdf/mid360_nanjing.urdf (robot description, URDF)
Before this commit: robot mid360, 8 links, 7 joints
Links:
- removed link fore_153
Joints:
- removed joint fore_153_joint

Commit message: feat: 20260123

File: src/cartographer_ros/cartographer_ros/urdf/mid360_nanjing.urdf (robot description, URDF)
Before this commit: robot mid360, 7 links, 6 joints
Links:
- added link wit_imu_link; visual box size=0.06 0.04 0.02
Joints:
- added joint wit_imu_link_joint: type fixed, parent base_link, child wit_imu_link, origin xyz=0 0 0.71325 rpy=0 0 0
